File: tecsci_dip/tecsci_dip/esp32_tmc5130.sch (KiCad schematic (older format))
At the start: 18 parts

Commit message: version 1.3
Parts:
- removed ?: AKL182_04_POL_HEADER, symbol TMC5130-Eval_v15-eagle-import:AKL182_04_POL_HEADER
- removed C? (x10): C, symbol Device:C
- removed D?: SMBJ, symbol TMC5130-Eval_v15-eagle-import:SMBJ
- removed R? (x3): R, symbol Device:R
Other:
- moved on the sheet: IC?
