File: tecsci_dip/tecsci_dip/esp32_tmc5130_.sch (KiCad schematic (older format))
At the start: 19 parts, among them IC201 TMC5130, J201 Conn_01x19_ESP32, J202 Conn_01x19_ESP32, U201 AKL182_04_POL_HEADER

Commit message: version 1.3
Parts:
- removed J201, J202: Conn_01x19_ESP32, Connector_PinSocket_2.54mm:PinSocket_1x19_P2.54mm_Vertical, symbol Connector_Generic:Conn_01x19
- added C211, C212: 0.1uF, Capacitor_SMD:C_0805_2012Metric, symbol Device:C
- added D202: PMEG3020CEH, Diode_SMD:D_SOD-123, symbol tecsci_dip-cache:PMEG6010CEH
- added J201: USB_B_Micro, Connector_USB:USB_Micro-B_Molex-105017-0001, symbol Connector:USB_B_Micro
- added J202: Boot, Connector_PinHeader_2.54mm:PinHeader_1x02_P2.54mm_Vertical, symbol Connector_Generic:Conn_01x02
- added J203: Conn_01x05, Connector_PinHeader_2.54mm:PinHeader_1x05_P2.54mm_Vertical, symbol Connector_Generic:Conn_01x05
- added J204: Conn_01x06, Connector_PinHeader_2.54mm:PinHeader_1x06_P2.54mm_Vertical, symbol Connector_Generic:Conn_01x06
- added Q201, Q202: S8050, Package_TO_SOT_SMD:SOT-23, symbol Transistor_BJT:S8050
- added R205, R206: 10K, Resistor_SMD:R_0805_2012Metric, symbol Device:R
- added R207: 4.7K, Resistor_SMD:R_0805_2012Metric, symbol Device:R
- added R208, R209: 1K, Resistor_SMD:R_0805_2012Metric, symbol Device:R
- added U202: ESP32-WROOM-32D, RF_Module:ESP32-WROOM-32, symbol RF_Module:ESP32-WROOM-32D
- added U203: CP2102N-A01-GQFN28, Package_DFN_QFN:QFN-28-1EP_5x5mm_P0.5mm_EP3.35x3.35mm, symbol Interface_USB:CP2102N-A01-GQFN28
- C201, C210: value 100uF -> 150uF/63V; digikey# (none) -> P15406-ND; manf (none) -> Panasonic Electronic Components; manf# (none) -> EEU-FR1J151
- C202, C206, C208: value 100nF -> 100nF/50V
- C203: value 470nF -> 470nF/16V
- C204: value 100nF -> 100nF/10V
- C205: value 4.7uF -> 4.7uF/16V
- C207: value 22nF -> 22nF/50V
- C209: value 4.7uF -> 4.7uF/100V
- R202, R204: value 0R15/0.5W -> 0R15
- U201: digikey# (none) -> 277-1208-ND
Connections:
- net +3V3: now also R207.2, U202.2 (VDD), U203.6 (VDD), U203.7 (REGIN); no longer C202.1, IC201.10 (VCC_IO)
- net +5VD: now also D202.1 (K)
- net CSN: now also U202.23 (IO15)
- net DRV_ENA: now also U202.27 (IO16)
- net GND: now also C211.2, C212.2, J201.5 (GND), J201.6 (Shield), J202.2 (Pin_2), U202.1 (GND), U202.15 (GND), U202.38 (GND), U203.29 (GND), U203.3 (GND)
- net MISO: now also U202.12 (IO27)
- net MOSI: now also U202.13 (IO14)
- net SCK: now also U202.14 (IO12)
- net CLK16: now reaches IC201.2 (CLK)
- new net: C202.1, IC201.10 (VCC_IO)
- new net: J204.2 (Pin_2), U202.10 (IO25)
- new net: J204.1 (Pin_1), U202.11 (IO26)
- new net: J203.1 (Pin_1), U202.28 (IO17)
- new net: J203.3 (Pin_3), U202.30 (IO18)
- new net: J203.4 (Pin_4), U202.31 (IO19)
- new net: J203.5 (Pin_5), U202.33 (IO21)
- new net: J204.6 (Pin_6), U202.6 (IO34)
- new net: J204.5 (Pin_5), U202.7 (IO35)
- new net: J204.4 (Pin_4), U202.8 (IO32)
- new net: J204.3 (Pin_3), U202.9 (IO33)
- new net: R208.2, U203.25 (RXD)
- new net: R209.2, U203.26 (TXD)
- new net: R207.1, U203.9 (~RSTb)
- new net: Q201.2 (B), R205.1
- new net: Q202.2 (B), R206.1
- new net D+: J201.3 (D+), U203.4 (D+)
- new net D-: J201.2 (D-), U203.5 (D-)
- new net DTR: Q202.1 (E), R205.2, U203.28 (~DTR)
- new net EN: C211.1, Q201.3 (C), U202.3 (EN)
- new net IO0: C212.1, J202.1 (Pin_1), Q202.3 (C), U202.25 (IO0)
- new net IO29: J203.2 (Pin_2), U202.29 (IO5)
- new net RTS: Q201.1 (E), R206.2, U203.24 (~RTS)
- new net RX: R209.1, U202.34 (RXD0/IO3)
- new net TX: R208.1, U202.35 (TXD0/IO1)
- new net VBUS: D202.2 (A), J201.1 (VBUS), U203.8 (VBUS)
- no-connect marks 40 -> 39
Other:
- note removed: "Módulo ESP32 NODEMCU v1.1"
