File: tecsci_dip/tecsci_dip/tecsci_dip.sch (KiCad schematic (older format))
At the start: 8 parts

Commit message: version 1.3
Changed lines of the file:
@@
 $EndDescr
 $Sheet
-S 2450 3850 2250 1550
+S 5250 1950 2250 1550
 U 5D952A19
 F0 "esp32_tmc5130_" 50
 F1 "esp32_tmc5130_.sch" 50
+F2 "CLK16" I L 5250 3150 50
 $EndSheet
 $Sheet
@@
 F0 "alimentacion" 50
 F1 "alimentacion.sch" 50
+F2 "CLK16" O R 4700 3150 50
 $EndSheet
 $Comp
@@
 	1    0    0    -1
 $EndComp
+Wire Wire Line
+	4700 3150 5250 3150
 $EndSCHEMATC
