File: tecsci_dip/tecsci_dip/alimentacion.sch (KiCad schematic (older format))
At the start: 16 parts, among them U301 Regulador_LM5161

Commit message: version 1.3
Parts:
- added C308: 10nF/16V/0805, Capacitor_SMD:C_0805_2012Metric, symbol Device:C
- added C310: 100nF, Capacitor_SMD:C_0805_2012Metric, symbol Device:C
- added C311: 10uF, Capacitor_SMD:C_0805_2012Metric, symbol Device:C
- added U302: LD1117S33TR_SOT223, Package_TO_SOT_SMD:SOT-223-3_TabPin2, symbol Regulator_Linear:LD1117S33TR_SOT223
- added X301: Oscillator_636L3C016M00000, Oscillator:Oscillator_SMD_EuroQuartz_XO53-4Pin_5.0x3.2mm, symbol Ponchobrücke-cache:Oscillator_636L3C016M00000
- D301: value PMEG6010CEH -> PMEG3020CEH; digikey# 1727-3848-2-ND -> 1727-3873-2-ND; manf# PMEG6010CEH,115 -> PMEG3020EH,115
- POWER_IN301: digikey# (none) -> 277-1106-ND
Connections:
- net +5VD: now also C310.1, U302.3 (VI)
- net GND: now also C308.2, C310.2, C311.2, U302.1 (GND), X301.2 (GND)
- net +5V: now reaches C306.1, C307.1, D301.2 (A), L301.2, R304.1
- new net: C308.1, X301.1 (EN)
- new net +3V3: C311.1, U302.2 (VO), X301.4 (Vcc)
- new net CLK16: X301.3 (OUT)
Other:
- note added: "Etapa Reguladora de Tensión\nEntrada 24-46Volt\nSalida 5V hacia integrado TMC130\nSalida 3.3V hacia microcontrolador con diodo de protección"
- note removed: "Etapa Reguladora de Tensión\nEntrada 24-46Volt\nSalida 5V hacia integrado TMC130\nSalida 5V hacia microcontrolador con diodo de protección"
- moved on the sheet: C301, C302, C303, C304, C305, C306, C307, D301, L301, POWER_IN301, R301, R302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

Commit message: version fabricada
Parts:
- C301: value 2.2uF -> 2.2uF/100V
- C302: value 100nF -> 100nF/100V
- C303: value 22nF -> 22nF/50V
- C304: value 1uF -> 1uF/50V
- C305: value 10nF -> 10nF/10V
- C306, C307, C311: value 10uF -> 10uF/10V
- C308: value 10nF/16V/0805 -> 10nF/16V
- C310: value 100nF -> 100nF/10V
- R301: value 30k -> 30k/1%; footprint Capacitor_SMD:C_0805_2012Metric -> Resistor_SMD:R_0805_2012Metric
- R302: value 6.8k -> 6.8k/1%
- R303: value 150k -> 150k/1%
- R304: value 3.3k -> 3.3k/1%
- R305: value 2.2k -> 2.2k/1%
Changed lines of the file:
@@
 P 3200 3150
 F 0 "C303" H 3315 3196 50  0000 L CNN
-F 1 "22nF" H 3315 3105 50  0000 L CNN
+F 1 "22nF/50V" H 3315 3105 50  0000 L CNN
 F 2 "Capacitor_SMD:C_0805_2012Metric" H 3238 3000 50  0001 C CNN
 F 3 "~" H 3200 3150 50  0001 C CNN
@@
 U 1 1 5D9C1E4A
 P 2050 3150
-F 0 "C302" H 2165 3196 50  0000 L CNN
-F 1 "100nF" H 2165 3105 50  0000 L CNN
+F 0 "C302" V 2100 2900 50  0000 L CNN
+F 1 "100nF/100V" V 2200 2900 50  0000 L CNN
 F 2 "Capacitor_SMD:C_1206_3216Metric" H 2088 3000 50  0001 C CNN
 F 3 "~" H 2050 3150 50  0001 C CNN
@@
 U 1 1 5D9C21D9
 P 1700 3150
-F 0 "C301" H 1815 3196 50  0000 L CNN
-F 1 "2.2uF" H 1815 3105 50  0000 L CNN
+F 0 "C301" V 1750 2900 50  0000 L CNN
+F 1 "2.2uF/100V" V 1850 2900 50  0000 L CNN
 F 2 "Capacitor_SMD:C_1206_3216Metric" H 1738 3000 50  0001 C CNN
 F 3 "~" H 1700 3150 50  0001 C CNN
@@
 P 5150 3150
 F 0 "C304" H 5265 3196 50  0000 L CNN
-F 1 "1uF" H 5265 3105 50  0000 L CNN
+F 1 "1uF/50V" H 5265 3105 50  0000 L CNN
 F 2 "Capacitor_SMD:C_0805_2012Metric" H 5188 3000 50  0001 C CNN
 F 3 "~" H 5150 3150 50  0001 C CNN
@@
 P 6750 3300
 F 0 "C306" H 6865 3346 50  0000 L CNN
-F 1 "10uF" H 6865 3255 50  0000 L CNN
+F 1 "10uF/10V" H 6865 3255 50  0000 L CNN
 F 2 "Capacitor_SMD:C_0805_2012Metric" H 6788 3150 50  0001 C CNN
 F 3 "~" H 6750 3300 50  0001 C CNN
@@
 P 7150 3300
 F 0 "C307" H 7265 3346 50  0000 L CNN
-F 1 "10uF" H 7265 3255 50  0000 L CNN
+F 1 "10uF/10V" H 7265 3255 50  0000 L CNN
 F 2 "Capacitor_SMD:C_0805_2012Metric" H 7188 3150 50  0001 C CNN
 F 3 "~" H 7150 3300 50  0001 C CNN
@@
 P 5300 2300
 F 0 "C305" V 5048 2300 50  0000 C CNN
-F 1 "10nF" V 5139 2300 50  0000 C CNN
+F 1 "10nF/10V" V 5139 2300 50  0000 C CNN
 F 2 "Capacitor_SMD:C_0805_2012Metric" H 5338 2150 50  0001 C CNN
 F 3 "~" H 5300 2300 50  0001 C CNN
@@
 U 1 1 5D9C42E9
 P 6350 2800
-F 0 "R304" H 6420 2846 50  0000 L CNN
-F 1 "3.3k" H 6420 2755 50  0000 L CNN
+F 0 "R304" H 6000 2850 50  0000 L CNN
+F 1 "3.3k/1%" H 6000 2750 50  0000 L CNN
 F 2 "Resistor_SMD:R_0805_2012Metric" V 6280 2800 50  0001 C CNN
 F 3 "~" H 6350 2800 50  0001 C CNN
@@
 U 1 1 5D9C7755
 P 6350 3300
-F 0 "R305" H 6420 3346 50  0000 L CNN
-F 1 "2.2k" H 6420 3255 50  0000 L CNN
+F 0 "R305" H 6050 3350 50  0000 L CNN
+F 1 "2.2k/1%" H 6000 3250 50  0000 L CNN
 F 2 "Resistor_SMD:R_0805_2012Metric" V 6280 3300 50  0001 C CNN
 F 3 "~" H 6350 3300 50  0001 C CNN
@@
 P 3100 2550
 F 0 "R303" V 2850 2550 50  0000 C CNN
-F 1 "150k" V 2950 2550 50  0000 C CNN
+F 1 "150k/1%" V 2950 2550 50  0000 C CNN
 F 2 "Resistor_SMD:R_0805_2012Metric" V 3030 2550 50  0001 C CNN
 F 3 "~" H 3100 2550 50  0001 C CNN
@@
 P 2500 2950
 F 0 "R301" H 2430 2904 50  0000 R CNN
-F 1 "30k" H 2430 2995 50  0000 R CNN
-F 2 "Capacitor_SMD:C_0805_2012Metric" V 2430 2950 50  0001 C CNN
+F 1 "30k/1%" H 2430 2995 50  0000 R CNN
+F 2 "Resistor_SMD:R_0805_2012Metric" V 2430 2950 50  0001 C CNN
 F 3 "~" H 2500 2950 50  0001 C CNN
 	1    2500 2950
@@
 P 2500 3450
 F 0 "R302" H 2430 3404 50  0000 R CNN
-F 1 "6.8k" H 2430 3495 50  0000 R CNN
+F 1 "6.8k/1%" H 2430 3495 50  0000 R CNN
 F 2 "Resistor_SMD:R_0805_2012Metric" V 2430 3450 50  0001 C CNN
 F 3 "~" H 2500 3450 50  0001 C CNN
@@
 P 1550 6200
 F 0 "C308" H 1350 6300 50  0000 L CNN
-F 1 "10nF/16V/0805" H 850 6150 50  0000 L CNN
+F 1 "10nF/16V" H 850 6150 50  0000 L CNN
 F 2 "Capacitor_SMD:C_0805_2012Metric" H 1588 6050 50  0001 C CNN
 F 3 "~" H 1550 6200 50  0001 C CNN
@@
 P 10700 3350
 F 0 "C311" H 10815 3396 50  0000 L CNN
-F 1 "10uF" H 10815 3305 50  0000 L CNN
+F 1 "10uF/10V" H 10815 3305 50  0000 L CNN
 F 2 "Capacitor_SMD:C_0805_2012Metric" H 10738 3200 50  0001 C CNN
 F 3 "~" H 10700 3350 50  0001 C CNN
@@
 P 9600 3350
 F 0 "C310" H 9715 3396 50  0000 L CNN
-F 1 "100nF" H 9715 3305 50  0000 L CNN
+F 1 "100nF/10V" H 9715 3305 50  0000 L CNN
 F 2 "Capacitor_SMD:C_0805_2012Metric" H 9638 3200 50  0001 C CNN
 F 3 "~" H 9600 3350 50  0001 C CNN
