File: tecsci_dip/tecsci_dip/tecsci_dip.kicad_pcb (KiCad board)
At the start: 2 copper layers, 65 x 60 mm, 43 parts, among them IC201 TMC5130, J201 Conn_01x19_ESP32, J202 Conn_01x19_ESP32, U201 AKL182_04_POL_HEADER, U301 Regulador_LM5161

Commit message: version 1.3
Parts:
- added C211: 0.1uF, Capacitor_SMD:C_0805_2012Metric, F.Cu at (58.8, 106.5)
- added C212: 0.1uF, Capacitor_SMD:C_0805_2012Metric, F.Cu at (68.4, 76.2)
- added C308: 10nF/16V/0805, Capacitor_SMD:C_0805_2012Metric, F.Cu at (86.4, 84.3)
- added C310: 100nF, Capacitor_SMD:C_0805_2012Metric, F.Cu at (82.6, 61.7)
- added C311: 10uF, Capacitor_SMD:C_0805_2012Metric, F.Cu at (72.5, 76.2)
- added D202: PMEG3020CEH, Diode_SMD:D_SOD-123, F.Cu at (79.4, 65.6)
- added J203: Conn_01x05, Connector_PinHeader_2.54mm:PinHeader_1x05_P2.54mm_Vertical, F.Cu at (75.4, 82.0)
- added J204: Conn_01x06, Connector_PinHeader_2.54mm:PinHeader_1x06_P2.54mm_Vertical, F.Cu at (78.0, 109.0)
- added Q201: S8050, Package_TO_SOT_SMD:SOT-23, F.Cu at (61.0, 64.4)
- added Q202: S8050, Package_TO_SOT_SMD:SOT-23, F.Cu at (61.0, 69.2)
- added R205: 10K, Resistor_SMD:R_0805_2012Metric, F.Cu at (65.5, 64.2)
- added R206: 10K, Resistor_SMD:R_0805_2012Metric, F.Cu at (65.4, 68.4)
- added R207: 4.7K, Resistor_SMD:R_0805_2012Metric, F.Cu at (72.5, 73.0)
- added R208: 1K, Resistor_SMD:R_0805_2012Metric, F.Cu at (61.0, 74.4)
- added R209: 1K, Resistor_SMD:R_0805_2012Metric, F.Cu at (68.4, 73.0)
- added U202: ESP32-WROOM-32D, RF_Module:ESP32-WROOM-32, F.Cu at (66.0, 95.5)
- added U203: CP2102N-A01-GQFN28, Package_DFN_QFN:QFN-28-1EP_5x5mm_P0.5mm_EP3.35x3.35mm, F.Cu at (71.4, 66.2)
- added U302: LD1117S33TR_SOT223, Package_TO_SOT_SMD:SOT-223-3_TabPin2, F.Cu at (79.8, 74.0)
- added X301: Oscillator_636L3C016M00000, Oscillator:Oscillator_SMD_EuroQuartz_XO53-4Pin_5.0x3.2mm, F.Cu at (85.2, 80.8)
- C201, C210: value 100uF -> 150uF/63V
- C202, C206, C208: value 100nF -> 100nF/50V
- C203: value 470nF -> 470nF/16V
- C204: value 100nF -> 100nF/10V
- C205: value 4.7uF -> 4.7uF/16V
- C207: value 22nF -> 22nF/50V
- C209: value 4.7uF -> 4.7uF/100V
- D301: value PMEG6010CEH -> PMEG3020CEH
- J201: value Conn_01x19_ESP32 -> USB_B_Micro; footprint Connector_PinSocket_2.54mm:PinSocket_1x19_P2.54mm_Vertical -> Connector_USB:USB_Micro-B_Molex-105017-0001
- J202: value Conn_01x19_ESP32 -> Boot; footprint Connector_PinSocket_2.54mm:PinSocket_1x19_P2.54mm_Vertical -> Connector_PinHeader_2.54mm:PinHeader_1x02_P2.54mm_Vertical
- R202, R204: value 0R15/0.5W -> 0R15
- moved J202 16.4 mm to (63.6, 77.6), turned to 270 degrees
- moved FID102 10.5 mm to (72.1, 112.3)
- moved J201 9.56 mm to (72.5, 58.8), turned to 180 degrees
- moved FID101 8.15 mm to (65.2, 58.4)
- moved H101 5.25 mm to (59.8, 111.2)
- moved H104 5.25 mm to (59.8, 58.8)
- moved FID103 0.95 mm to (117.2, 65.6)
Connections:
- net Net-(C306-Pad1) renamed +5V
- C202 pad 1: +3V3 -> Net-(C202-Pad1)
- IC201 pad 10: +3V3 -> Net-(C202-Pad1)
- IC201 pad 2: Net-(IC201-Pad2) -> /alimentacion/CLK16
- J201 pad 1: +5VD -> /esp32_tmc5130_/VBUS
- J201 pad 2: Net-(J201-Pad2) -> /esp32_tmc5130_/D-
- J201 pad 3: Net-(J201-Pad3) -> /esp32_tmc5130_/D+
- J201 pad 5: Net-(J201-Pad5) -> GND
- J201 pad 6: Net-(J201-Pad6) -> GND
- J202 pad 1: Net-(J202-Pad1) -> /esp32_tmc5130_/IO0
- J202 pad 2: Net-(J202-Pad2) -> GND
Routing:
- net GND: track 211.6 -> 292.2 mm, vias 1 -> 9
- net /esp32_tmc5130_/EN: track 0.00 -> 44.9 mm, vias 0 -> 2
- net +3V3: track 31.7 -> 69.1 mm, vias 0 -> 2
- net /esp32_tmc5130_/IO0: track 0.00 -> 34.6 mm, vias 0 -> 2
- net /esp32_tmc5130_/DTR: track 0.00 -> 29.1 mm, vias 0 -> 2
- net /esp32_tmc5130_/MISO: track 16.0 -> 36.7 mm, vias 1 -> 0
- net /esp32_tmc5130_/CSN: track 42.6 -> 22.0 mm, vias 1 -> 0
- net /esp32_tmc5130_/MOSI: track 16.6 -> 35.5 mm, vias 1 -> 0
- net /esp32_tmc5130_/RX: track 0.00 -> 15.9 mm, vias 0 -> 2
- net /esp32_tmc5130_/SCK: track 16.9 -> 32.6 mm, vias 1 -> 0
- net /esp32_tmc5130_/DRV_ENA: track 53.8 -> 38.9 mm, vias 1 -> 2
- net /esp32_tmc5130_/VBUS: track 0.00 -> 14.8 mm
- net Net-(R208-Pad2): track 0.00 -> 14.2 mm, vias 0 -> 2
- net /esp32_tmc5130_/TX: track 0.00 -> 14.1 mm
- net +5VD: track 3.45 -> 17.4 mm
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Other:
- board text added: "Grilla de posicionamiento: Principal 0,25mm Grilla de ruteo: Principal 0,25mm Mounting Hole: Principal: 3,2mm Pistas: Principal 0.5mm Alternativa inferior 0.25mm (Límite Mayer 8mils - 0.20mm) Alternativa superior 0,8mm Vías: Principal 0.8mm/0.4mm (Límite Mayer 8mils - 32(0.8mm)-16(0.4mm) ) Margen General : 0,22 mm Margen Particular: 0,2 mm Componentes -> 201 301 (Límite Mayer 8mils - 0.18mm) Base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"
- board text added: "TECSCI https://tecsci.com.ar"
- board text added: "Technology for Science Dip Coater v1.3"
- board text removed: "Grilla de posicionamiento: Principal 0,25mm Grilla de ruteo: Principal 0,25mm Mounting Hole: Principal: 3,2mm Pistas: Principal 0.5mm Alternativa inferior 0.25mm (Límite Mayer 8mils - 0.20mm) Alternativa superior 0,8mm Vías: Principal 0.8mm/0.4mm (Límite Mayer 8mils - 0.80mm) Margen General : 0,22 mm Margen Particular: 0,2 mm Componentes -> 201 301 (Límite Mayer 8mils - 0.18mm) Base para las rest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"
- board text removed: "TECSCI"
- board text removed: "TecSci Tecnología para Ciencia Dip Coater v1.0"
- board text removed: "https://tecsci.com.ar/"

Commit message: version fabricada
Parts:
- C204: value 100nF/10V -> 100nF/50V
- C211, C212: value 0.1uF -> 0.1uF/10V
- C301: value 2.2uF -> 2.2uF/100V
- C302: value 100nF -> 100nF/100V
- C303: value 22nF -> 22nF/50V
- C304: value 1uF -> 1uF/50V
- C305: value 10nF -> 10nF/10V
- C306, C307, C311: value 10uF -> 10uF/10V
- C308: value 10nF/16V/0805 -> 10nF/16V
- C310: value 100nF -> 100nF/10V
- R201: value 2R2 -> 2R2/1%
- R202, R204: value 0R15 -> 0R15/1%
- R203: value 0R -> 0R/1%
- R205, R206: value 10K -> 10K/1%
- R207: value 4.7K -> 4.7K/1%
- R208, R209: value 1K -> 1K/1%
- R301: value 30k -> 30k/1%; footprint Capacitor_SMD:C_0805_2012Metric -> Resistor_SMD:R_0805_2012Metric
- R302: value 6.8k -> 6.8k/1%
- R303: value 150k -> 150k/1%
- R304: value 3.3k -> 3.3k/1%
- R305: value 2.2k -> 2.2k/1%
Connections:
- C202 pad 1: Net-(C202-Pad1) -> +3V3
- IC201 pad 10: Net-(C202-Pad1) -> +3V3
- U202 pad 39: GND -> (no net)
Routing:
- net +3V3: track 69.1 -> 95.9 mm, vias 2 -> 4
- net Net-(C202-Pad1): track 9.00 -> 0.00 mm
